File: Bluetooth-Speaker-KiCad/Bluetooth-Speaker-KiCad.kicad_pcb (KiCad board)
At the start: 4 copper layers, 42 x 41 mm, 36 parts, among them J1 USB4105-GF-A, J2 Screw_Terminal_01x02, J3 Screw_Terminal_01x02, Q1 Q_PMOS_DSG, U1 TPD4E02B04DQA, U2 MAX1811, U3 RT6150B-33GQW, U5 ESP32-C3-WROOM-02, U6 MAX98357A

Commit message: Updated final PCB render
Other:
- board text added: "PCB3D_BR_BluetoothSpeaker"
- board text added: "PCB3D_TL_BluetoothSpeaker"
Changed lines of the file:
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@@
 		(tags "capacitor handsolder")
 		(property "Reference" "C11"
-			(at 0 -1.43 360)
+			(at 0 -1.43 0)
 			(layer "F.SilkS")
 			(effects
@@
 		)
 		(property "Value" "0.1u"
-			(at 0 1.43 360)
+			(at 0 1.43 0)
 			(layer "F.Fab")
 			(effects
@@
 		)
 		(fp_text user "${REFERENCE}"
-			(at 0 0 360)
+			(at 0 0 0)
 			(layer "F.Fab")
 			(effects
@@
 		(at 130.73 111.78 180)
 		(property "Reference" "S2"
-			(at -0.985855 -1.455943 360)
+			(at -0.985855 -1.455943 0)
 			(layer "F.SilkS")
 			(effects
@@
 		)
 		(property "Value" "EVP-AWCD4A"
-			(at 0.643575 1.551574 360)
+			(at 0.643575 1.551574 0)
 			(layer "F.Fab")
 			(effects
@@
 		)
 		(property "Footprint" "EVP_AWCD4A (1):SW_EVP-AWCD4A"
-			(at 0 0 360)
+			(at 0 0 0)
 			(layer "F.Fab")
 			(hide yes)
@@
 		)
 		(property "Datasheet" ""
-			(at 0 0 360)
+			(at 0 0 0)
 			(layer "F.Fab")
 			(hide yes)
@@
 		)
 		(property "Description" ""
-			(at 0 0 360)
+			(at 0 0 0)
 			(layer "F.Fab")
 			(hide yes)
@@
 		(tags "capacitor handsolder")
 		(property "Reference" "C10"
-			(at 0.0075 -1.42 360)
+			(at 0.0075 -1.42 0)
 			(layer "F.SilkS")
 			(effects
@@
 		)
 		(property "Value" "0.1u"
-			(at 0 1.43 360)
+			(at 0 1.43 0)
 			(layer "F.Fab")
 			(effects
@@
 		)
 		(fp_text user "${REFERENCE}"
-			(at 0 0 360)
+			(at 0 0 0)
 			(layer "F.Fab")
 			(effects
@@
 		(layer "Edge.Cuts")
 	)
+	(gr_text "PCB3D_BR_BluetoothSpeaker"
+		(at 169.59 147.38 0)
+		(layer "In2.Cu")
+		(effects
+			(font
+				(size 1.5 1.5)
+				(thickness 0.3)
+				(bold yes)
+			)
+			(justify left bottom)
+		)
+	)
+	(gr_text "PCB3D_TL_BluetoothSpeaker"
+		(at 119.95 86.93 0)
+		(layer "In2.Cu")
+		(effects
+			(font
+				(size 1.5 1.5)
+				(thickness 0.3)
+				(bold yes)
+			)
+			(justify left bottom)
+		)
+	)
 	(segment
